Commit message: using gazebo ignition

File: models/robots/mir100/urdf/include/common.gazebo.xacro (robot description, xacro)
@@ -2,13 +2,38 @@
 <robot xmlns:xacro="http://ros.org/wiki/xacro">
   <xacro:macro name="controller_plugin_gazebo" params="robot_namespace">
-    <gazebo>
-      <plugin name="gazebo_ros_control" filename="libgazebo_ros_control.so">
-        <xacro:unless value="${robot_namespace == ''}">
-          <robotNamespace>${robot_namespace}</robotNamespace>
-        </xacro:unless>
-        <controlPeriod>0.001</controlPeriod>
-        <legacyModeNS>false</legacyModeNS>
-      </plugin>
-    </gazebo>
+    <xacro:if value="${gazebo_version == 'classic'}">
+      <gazebo>
+        <plugin name="gazebo_ros_control" filename="libgazebo_ros_control.so">
+          <xacro:unless value="${robot_namespace == ''}">
+            <robotNamespace>${robot_namespace}</robotNamespace>
+          </xacro:unless>
+          <controlPeriod>0.001</controlPeriod>
+          <legacyModeNS>false</legacyModeNS>
+        </plugin>
+      </gazebo>
+    </xacro:if>
+    <xacro:if value="${gazebo_version == 'ignition'}">
+      <ros2_control name="IgnitionSystem" type="system">
+        <hardware>
+          <plugin>ign_ros2_control/IgnitionSystem</plugin>
+        </hardware>
+        <joint name="${prefix}left_wheel_joint">
+          <command_interface name="velocity">
+            <param name="min">-1</param>
+            <param name="max">1</param>
+          </command_interface>
+          <state_interface name="position"/>
+          <state_interface name="velocity"/>
+        </joint>
+        <joint name="${prefix}right_wheel_joint">
+          <command_interface name="velocity">
+            <param name="min">-1</param>
+            <param name="max">1</param>
+          </command_interface>
+          <state_interface name="position"/>
+          <state_interface name="velocity"/>
+        </joint>
+      </ros2_control>
+    </xacro:if>
   </xacro:macro>
 </robot>

File: models/robots/mir100/urdf/include/imu.gazebo.urdf.xacro (robot description, xacro)
@@ -18,13 +18,15 @@
         <visualize>true</visualize>
         <topic>__default_topic__</topic>
-        <plugin filename="libgazebo_ros_imu_sensor.so" name="imu_plugin">
-          <topicName>${imu_topic}</topicName>
-          <bodyName>${link}</bodyName>
-          <updateRateHZ>${update_rate}</updateRateHZ>  <!-- this is the publish rate -->
-          <gaussianNoise>${stdev * stdev}</gaussianNoise>
-          <xyzOffset>0 0 0</xyzOffset>
-          <rpyOffset>0 0 0</rpyOffset>
-          <frameName>${imu_frame}</frameName>  <!-- from real MiR -->
-        </plugin>
+        <xacro:if value="${gazebo_version == 'classic'}">
+          <plugin filename="libgazebo_ros_imu_sensor.so" name="imu_plugin">
+            <topicName>${imu_topic}</topicName>
+            <bodyName>${link}</bodyName>
+            <updateRateHZ>${update_rate}</updateRateHZ>  <!-- this is the publish rate -->
+            <gaussianNoise>${stdev * stdev}</gaussianNoise>
+            <xyzOffset>0 0 0</xyzOffset>
+            <rpyOffset>0 0 0</rpyOffset>
+            <frameName>${imu_frame}</frameName>  <!-- from real MiR -->
+          </plugin>
+        </xacro:if>
         <pose>0 0 0 0 0 0</pose>
       </sensor>

File: models/robots/mir100/urdf/include/mir_100.gazebo.xacro (robot description, xacro)
@@ -3,24 +3,34 @@
   <xacro:macro name="diff_controller_plugin_gazebo" params="prefix left_wheel_joint right_wheel_joint wheel_separation wheel_radius">
     <gazebo>
-      <plugin name="diff_drive_controller" filename="libgazebo_ros_diff_drive.so">
-        <legacyMode>false</legacyMode>
-        <alwaysOn>true</alwaysOn>
-        <updateRate>1000.0</updateRate>
-        <leftJoint>${left_wheel_joint}</leftJoint>
-        <rightJoint>${right_wheel_joint}</rightJoint>
-        <wheelSeparation>${wheel_separation}</wheelSeparation>
-        <wheelDiameter>${2*wheel_radius}</wheelDiameter>
-        <wheelTorque>10</wheelTorque>
-        <publishTf>1</publishTf>
-        <odometryFrame>map</odometryFrame>
-        <commandTopic>mobile_base_controller/cmd_vel</commandTopic>
-        <odometryTopic>mobile_base_controller/odom</odometryTopic>
-        <robotBaseFrame>base_footprint</robotBaseFrame>
-        <wheelAcceleration>2.8</wheelAcceleration>
-        <publishWheelJointState>true</publishWheelJointState>
-        <publishWheelTF>false</publishWheelTF>
-        <odometrySource>world</odometrySource>
-        <rosDebugLevel>Debug</rosDebugLevel>
-      </plugin>
+      <xacro:if value="${gazebo_version == 'classic'}">
+        <plugin name="diff_drive_controller" filename="libgazebo_ros_diff_drive.so">
+          <legacyMode>false</legacyMode>
+          <alwaysOn>true</alwaysOn>
+          <updateRate>1000.0</updateRate>
+          <leftJoint>${left_wheel_joint}</leftJoint>
+          <rightJoint>${right_wheel_joint}</rightJoint>
+          <wheelSeparation>${wheel_separation}</wheelSeparation>
+          <wheelDiameter>${2*wheel_radius}</wheelDiameter>
+          <wheelTorque>10</wheelTorque>
+          <publishTf>1</publishTf>
+          <odometryFrame>map</odometryFrame>
+          <commandTopic>mobile_base_controller/cmd_vel</commandTopic>
+          <odometryTopic>mobile_base_controller/odom</odometryTopic>
+          <robotBaseFrame>base_footprint</robotBaseFrame>
+          <wheelAcceleration>2.8</wheelAcceleration>
+          <publishWheelJointState>true</publishWheelJointState>
+          <publishWheelTF>false</publishWheelTF>
+          <odometrySource>world</odometrySource>
+          <rosDebugLevel>Debug</rosDebugLevel>
+        </plugin>
+      </xacro:if>
+      <xacro:if value="${gazebo_version == 'ignition'}">
+        <plugin filename="ign_ros2_control-system" name="ign_ros2_control::IgnitionROS2ControlPlugin">
+          <ros>
+            <namespace>/$(arg model_name)</namespace>
+          </ros>
+          <parameters>$(find senai_models)/models/${model_class}/${model}/config/$(arg gazebo_version)/${model}_controllers.yaml</parameters>
+        </plugin>
+      </xacro:if>
     </gazebo>
   </xacro:macro>
@@ -44,14 +54,16 @@
   <xacro:macro name="p3d_base_controller" params="prefix">
     <gazebo>
-      <plugin name="p3d_base_controller" filename="libgazebo_ros_p3d.so">
-        <alwaysOn>true</alwaysOn>
-        <updateRate>50.0</updateRate>
-        <bodyName>${prefix}base_footprint</bodyName>
-        <topicName>base_pose_ground_truth</topicName>
-        <gaussianNoise>0.01</gaussianNoise>
-        <frameName>map</frameName>
-        <xyzOffsets>0 0 0</xyzOffsets>
-        <rpyOffsets>0 0 0</rpyOffsets>
-      </plugin>
+      <xacro:if value="${gazebo_version == 'classic'}">
+        <plugin name="p3d_base_controller" filename="libgazebo_ros_p3d.so">
+          <alwaysOn>true</alwaysOn>
+          <updateRate>50.0</updateRate>
+          <bodyName>${prefix}base_footprint</bodyName>
+          <topicName>base_pose_ground_truth</topicName>
+          <gaussianNoise>0.01</gaussianNoise>
+          <frameName>map</frameName>
+          <xyzOffsets>0 0 0</xyzOffsets>
+          <rpyOffsets>0 0 0</rpyOffsets>
+        </plugin>
+      </xacro:if>
     </gazebo>
   </xacro:macro>

File: models/robots/mir100/urdf/include/sick_s300.urdf.xacro (robot description, xacro)
@@ -56,8 +56,10 @@
           </noise>
         </ray>
-        <plugin name="gazebo_ros_${link}_controller" filename="libgazebo_ros_laser.so">
-          <frameName>${prefix}${link}</frameName>
-          <topicName>${topic}</topicName>
-        </plugin>
+        <xacro:if value="${gazebo_version == 'classic'}">
+          <plugin name="gazebo_ros_${link}_controller" filename="libgazebo_ros_laser.so">
+            <frameName>${prefix}${link}</frameName>
+            <topicName>${topic}</topicName>
+          </plugin>
+        </xacro:if>
       </sensor>
     </gazebo>

File: models/robots/mir100/urdf/mir100.urdf.xacro (robot description, xacro)
@@ -1,5 +1,7 @@
 <?xml version="1.0"?>
 <robot xmlns:xacro="http://ros.org/wiki/xacro" name="$(arg model_name)" >
+  <xacro:arg name="gazebo_version" default="ignition" />
   <xacro:arg name="model_name" default="bot" />
+  <xacro:property name="gazebo_version" value="$(arg gazebo_version)"/>
   <xacro:property name="model_class" value="robots" />
   <xacro:property name="model" value="mir100" />
@@ -16,11 +18,11 @@
   </xacro:unless>
   <xacro:mir_100 prefix="${prefix}"/>
-  <xacro:controller_plugin_gazebo robot_namespace=""/>
-  <!-- instead of the controller_plugin_gazebo, you can use the diffdrive controller like this:
-    <xacro:diff_controller_plugin_gazebo prefix=""
-      left_wheel_joint="left_wheel_joint"
-      right_wheel_joint="right_wheel_joint"
-      wheel_separation="${2*mir_100_act_wheel_dy}"
-      wheel_radius="${mir_100_act_wheel_radius}"/>
-  -->
+  <xacro:controller_plugin_gazebo robot_namespace="$(arg model_name)"/>
+  <!-- instead of the controller_plugin_gazebo, you can use the diffdrive controller like this:-->
+  <xacro:diff_controller_plugin_gazebo prefix=""
+    left_wheel_joint="left_wheel_joint"
+    right_wheel_joint="right_wheel_joint"
+    wheel_separation="${2*mir_100_act_wheel_dy}"
+    wheel_radius="${mir_100_act_wheel_radius}"
+  />
 </robot>
