Commit message: fixing diff_drive for gazebo classic, working on ignition

File: models/robots/mir100/urdf/include/common.gazebo.xacro (robot description, xacro)
@@ -13,39 +13,4 @@
       </gazebo>
     </xacro:if>
-    <xacro:if value="${gazebo_version == 'ignition'}">
-      <ros2_control name="IgnitionSystem" type="system">
-        <hardware>
-          <plugin>ign_ros2_control/IgnitionSystem</plugin>
-        </hardware>
-        <joint name="${prefix}left_wheel_joint">
-          <command_interface name="velocity">
-            <param name="min">-1</param>
-            <param name="max">1</param>
-          </command_interface>
-          <state_interface name="position"/>
-          <state_interface name="velocity"/>
-        </joint>
-        <joint name="${prefix}right_wheel_joint">
-          <command_interface name="velocity">
-            <param name="min">-1</param>
-            <param name="max">1</param>
-          </command_interface>
-          <state_interface name="position"/>
-          <state_interface name="velocity"/>
-        </joint>
-        <sensor name="imu_sensor">
-          <state_interface name="orientation.x" />
-          <state_interface name="orientation.y" />
-          <state_interface name="orientation.z" />
-          <state_interface name="orientation.w" />
-          <state_interface name="angular_velocity.x" />
-          <state_interface name="angular_velocity.y" />
-          <state_interface name="angular_velocity.z" />
-          <state_interface name="linear_acceleration.x" />
-          <state_interface name="linear_acceleration.y" />
-          <state_interface name="linear_acceleration.z" />
-        </sensor>
-      </ros2_control>
-    </xacro:if>
   </xacro:macro>
 </robot>

File: models/robots/mir100/urdf/include/imu.gazebo.urdf.xacro (robot description, xacro)
@@ -17,5 +17,5 @@
         <update_rate>100</update_rate>  <!-- this is not the publish rate -->
         <visualize>true</visualize>
-        <topic>__default_topic__</topic>
+        <topic>/model/$(arg model_name)/imu_data</topic>
         <plugin filename="ignition-gazebo-imu-system" name="gz::sim::systems::Imu">
           <topicName>${imu_topic}</topicName>

File: models/robots/mir100/urdf/include/mir_100.gazebo.xacro (robot description, xacro)
@@ -15,6 +15,6 @@
           <publishTf>1</publishTf>
           <odometryFrame>map</odometryFrame>
-          <commandTopic>mobile_base_controller/cmd_vel</commandTopic>
-          <odometryTopic>mobile_base_controller/odom</odometryTopic>
+          <commandTopic>/model/$(arg model_name)/cmd_vel</commandTopic>
+          <odometryTopic>/model/$(arg model_name)/odom</odometryTopic>
           <robotBaseFrame>base_footprint</robotBaseFrame>
           <wheelAcceleration>2.8</wheelAcceleration>
@@ -26,15 +26,19 @@
       </xacro:if>
       <xacro:if value="${gazebo_version == 'ignition'}">
-        <plugin filename="ignition-gazebo-diff-drive-system" name="gz::sim::systems::DiffDrive">
+        <plugin filename="gz-sim-diff-drive-system" name="gz::sim::systems::DiffDrive">
           <left_joint>${left_wheel_joint}</left_joint>
           <right_joint>${right_wheel_joint}</right_joint>
-          <wheel_separation>${wheel_separation}</wheel_separation>
-          <wheel_radius>${wheel_radius}</wheel_radius>
-          <!--
-          <topic>/cmd_vel</topic>
-          <odom_topic>/odom</odom_topic>
-          <odom_publish_frequency>1</odom_publish_frequency>
-          -->
+          <!-- <wheel_separation>${wheel_separation}</wheel_separation>
+          <wheel_radius>${wheel_radius}</wheel_radius> -->
+          <wheel_separation>0.445</wheel_separation>
+          <wheel_radius>0.06</wheel_radius>
           <max_linear_acceleration>2.0</max_linear_acceleration>
+          <topic>/model/$(arg model_name)/cmd_vel</topic>
+          <odom_topic>/model/$(arg model_name)/odom</odom_topic>
+          <tf_topic>/model/$(arg model_name)/tf</tf_topic>
+          <frame_id>odom</frame_id>
+          <child_frame_id>base_footprint</child_frame_id>
+          <odom_publish_frequency>30</odom_publish_frequency>
+          <!-- <max_linear_acceleration>2.0</max_linear_acceleration>
           <min_linear_acceleration>-2.0</min_linear_acceleration>
           <max_angular_acceleration>2.5</max_angular_acceleration>
@@ -43,5 +47,5 @@
           <min_linear_velocity>-1.0</min_linear_velocity>
           <max_angular_velocity>1.5</max_angular_velocity>
-          <min_angular_velocity>-1.5</min_angular_velocity>
+          <min_angular_velocity>-1.5</min_angular_velocity> -->
         </plugin>
       </xacro:if>
@@ -66,6 +70,6 @@
   </xacro:macro>
   <xacro:macro name="p3d_base_controller" params="prefix">
-    <gazebo>
-      <xacro:if value="${gazebo_version == 'classic'}">
+    <xacro:if value="${gazebo_version == 'classic'}">
+      <gazebo>
         <plugin name="p3d_base_controller" filename="libgazebo_ros_p3d.so">
           <alwaysOn>true</alwaysOn>
@@ -78,8 +82,8 @@
           <rpyOffsets>0 0 0</rpyOffsets>
         </plugin>
-      </xacro:if>
-      <xacro:if value="${gazebo_version == 'ignition'}">
-      </xacro:if>
-    </gazebo>
+      </gazebo>
+    </xacro:if>
+    <xacro:if value="${gazebo_version == 'ignition'}">
+    </xacro:if>
   </xacro:macro>
 </robot>

File: models/robots/mir100/urdf/include/mir_100_v1.urdf.xacro (robot description, xacro)
@@ -3,5 +3,5 @@
   <xacro:include filename="$(find senai_models)/models/${model_class}/${model}/urdf/include/common_properties.urdf.xacro" />
   <xacro:include filename="$(find senai_models)/models/${model_class}/${model}/urdf/include/imu.gazebo.urdf.xacro" />
-  <xacro:include filename="$(find senai_models)/models/${model_class}/${model}/urdf/include/mir_100.gazebo.xacro" />
+  <!-- <xacro:include filename="$(find senai_models)/models/${model_class}/${model}/urdf/include/mir_100.gazebo.xacro" /> -->
   <xacro:include filename="$(find senai_models)/models/${model_class}/${model}/urdf/include/mir_100.transmission.xacro" />
   <xacro:include filename="$(find senai_models)/models/${model_class}/${model}/urdf/include/sick_s300.urdf.xacro" />

File: models/robots/mir100/urdf/include/sick_s300.urdf.xacro (robot description, xacro)
@@ -29,7 +29,46 @@
       <!-- <material value="Gazebo/Yellow" /> -->
       <material value="Gazebo/FlatBlack" />
-      <sensor type="ray" name="${prefix}${link}">
+      <sensor name="${prefix}${link}" type='lidar'>
         <pose>0 0 0 0 0 0</pose>
-        <visualize>false</visualize>
+        <visualize>true</visualize>
+        <update_rate>12.5</update_rate>
+        <lidar>
+            <scan>
+                <horizontal>
+                    <samples>541</samples>
+                    <resolution>1</resolution>
+                    <min_angle>-2.35619449615</min_angle>
+                    <max_angle>2.35619449615</max_angle>
+                </horizontal>
+            </scan>
+            <range>
+                <min>0.05</min>
+                <max>29.0</max>
+                <resolution>0.01</resolution>
+            </range>
+            <noise>
+              <type>gaussian</type>
+              <!-- Noise parameters based on published spec for S300 achieving
+                  "+-29mm" accuracy at range < 3m (~0.01 of the range) at
+                  1 sigma. -->
+              <mean>0.0</mean>
+              <stddev>0.01</stddev>
+            </noise>
+        </lidar>
+        <xacro:if value="${gazebo_version == 'classic'}">
+          <plugin name="gazebo_ros_${link}_controller" filename="libgazebo_ros_laser.so">
+            <frameName>${prefix}${link}</frameName>
+            <topicName>${topic}</topicName>
+          </plugin>
+        </xacro:if>
+        <xacro:if value="${gazebo_version == 'ignition'}">
+          <plugin filename="libignition-gazebo-sensors-system.so" name="ignition::gazebo::systems::Sensors">
+            <render_engine>ogre2</render_engine>
+          </plugin>
+        </xacro:if>
+      </sensor>
+      <!-- <sensor type="ray" name="${prefix}${link}">
+        <pose>0 0 0 0 0 0</pose>
+        <visualize>true</visualize>
         <update_rate>12.5</update_rate>
         <ray>
@@ -37,5 +76,5 @@
             <horizontal>
               <samples>541</samples>
-              <resolution>1</resolution>  <!-- has to be 1; actual resolution will be computed from number of samples + min_angle/max_angle -->
+              <resolution>1</resolution>  <!- has to be 1; actual resolution will be computed from number of samples + min_angle/max_angle ->
               <min_angle>-2.35619449615</min_angle>
               <max_angle>2.35619449615</max_angle>
@@ -49,7 +88,7 @@
           <noise>
             <type>gaussian</type>
-            <!-- Noise parameters based on published spec for S300 achieving
+            <!- Noise parameters based on published spec for S300 achieving
                  "+-29mm" accuracy at range < 3m (~0.01 of the range) at
-                 1 sigma. -->
+                 1 sigma. ->
             <mean>0.0</mean>
             <stddev>0.01</stddev>
@@ -62,5 +101,5 @@
           </plugin>
         </xacro:if>
-      </sensor>
+      </sensor> -->
     </gazebo>
   </xacro:macro>

File: models/robots/mir100/urdf/mir100.urdf.xacro (robot description, xacro)
@@ -8,5 +8,5 @@
   <!-- MiR100 base -->
   <xacro:include filename="$(find senai_models)/models/${model_class}/${model}/urdf/include/mir_100_v1.urdf.xacro" />
-  <xacro:include filename="$(find senai_models)/models/${model_class}/${model}/urdf/include/common.gazebo.xacro" />
+  <!-- <xacro:include filename="$(find senai_models)/models/${model_class}/${model}/urdf/include/common.gazebo.xacro" /> -->
   <xacro:arg name="tf_prefix" default="" />
   <xacro:property name="tf_prefix_" value="$(arg tf_prefix)" />
@@ -18,19 +18,98 @@
   </xacro:unless>
   <xacro:mir_100 prefix="${prefix}"/>
-  <xacro:controller_plugin_gazebo robot_namespace="$(arg model_name)"/>
+  <!-- <xacro:controller_plugin_gazebo robot_namespace="$(arg model_name)"/> -->
   <!-- instead of the controller_plugin_gazebo, you can use the diffdrive controller like this:-->
-  <xacro:diff_controller_plugin_gazebo prefix=""
+  <!-- <xacro:diff_controller_plugin_gazebo prefix=""
     left_wheel_joint="left_wheel_joint"
     right_wheel_joint="right_wheel_joint"
     wheel_separation="${2*mir_100_act_wheel_dy}"
     wheel_radius="${mir_100_act_wheel_radius}"
-  />
-  <gazebo>
-    <plugin filename="ign_ros2_control-system" name="ign_ros2_control::IgnitionROS2ControlPlugin">
-      <ros>
-        <namespace>/$(arg model_name)</namespace>
-      </ros>
-      <parameters>$(find senai_models)/models/${model_class}/${model}/config/$(arg gazebo_version)/${model}_controllers.yaml</parameters>
-    </plugin>
-  </gazebo>
+  /> -->
+  <!-- ros2_control parameters: -->
+  <xacro:if value="${gazebo_version == 'classic'}">
+    <ros2_control name="GazeboSystem" type="system">
+      <hardware>
+        <plugin>gazebo_ros2_control/GazeboSystem</plugin>
+      </hardware>
+      <joint name="left_wheel_joint">
+        <command_interface name="velocity">
+            <param name="min">-10</param>
+            <param name="max">10</param>
+        </command_interface>
+        <state_interface name="position" />
+        <state_interface name="velocity" />
+      </joint>
+      <joint name="right_wheel_joint">
+          <command_interface name="velocity">
+              <param name="min">-10</param>
+              <param name="max">10</param>
+          </command_interface>
+          <state_interface name="velocity" />
+          <state_interface name="position" />
+      </joint>
+      <sensor name="imu_sensor">
+        <state_interface name="orientation.x" />
+        <state_interface name="orientation.y" />
+        <state_interface name="orientation.z" />
+        <state_interface name="orientation.w" />
+        <state_interface name="angular_velocity.x" />
+        <state_interface name="angular_velocity.y" />
+        <state_interface name="angular_velocity.z" />
+        <state_interface name="linear_acceleration.x" />
+        <state_interface name="linear_acceleration.y" />
+        <state_interface name="linear_acceleration.z" />
+      </sensor>
+    </ros2_control>
+    <gazebo>
+      <plugin filename="libgazebo_ros2_control.so" name="gazebo_ros2_control">
+        <ros>
+          <namespace>/$(arg model_name)</namespace>
+        </ros>
+        <parameters>$(find senai_models)/models/${model_class}/${model}/config/$(arg gazebo_version)/${model}_controllers.yaml</parameters>
+      </plugin>
+    </gazebo>
+  </xacro:if>
+  <xacro:if value="${gazebo_version == 'ignition'}">
+    <ros2_control name="IgnitionSystem" type="system">
+      <hardware>
+        <plugin>ign_ros2_control/IgnitionSystem</plugin>
+      </hardware>
+      <joint name="left_wheel_joint">
+        <command_interface name="velocity">
+            <param name="min">-10</param>
+            <param name="max">10</param>
+        </command_interface>
+        <state_interface name="position" />
+        <state_interface name="velocity" />
+      </joint>
+      <joint name="right_wheel_joint">
+          <command_interface name="velocity">
+              <param name="min">-10</param>
+              <param name="max">10</param>
+          </command_interface>
+          <state_interface name="velocity" />
+          <state_interface name="position" />
+      </joint>
+      <sensor name="imu_sensor">
+        <state_interface name="orientation.x" />
+        <state_interface name="orientation.y" />
+        <state_interface name="orientation.z" />
+        <state_interface name="orientation.w" />
+        <state_interface name="angular_velocity.x" />
+        <state_interface name="angular_velocity.y" />
+        <state_interface name="angular_velocity.z" />
+        <state_interface name="linear_acceleration.x" />
+        <state_interface name="linear_acceleration.y" />
+        <state_interface name="linear_acceleration.z" />
+      </sensor>
+    </ros2_control>
+    <gazebo>
+      <plugin filename="ign_ros2_control-system" name="ign_ros2_control::IgnitionROS2ControlPlugin">
+        <ros>
+          <namespace>/$(arg model_name)</namespace>
+        </ros>
+        <parameters>$(find senai_models)/models/${model_class}/${model}/config/$(arg gazebo_version)/${model}_controllers.yaml</parameters>
+      </plugin>
+    </gazebo>
+  </xacro:if>
 </robot>
