Commit message: fixing mir100 model import, error while using rviz2

File: models/robots/mir100/urdf/include/mir_100_v1.urdf.xacro (robot description, xacro)
@@ -1,9 +1,9 @@
 <?xml version="1.0"?>
 <robot xmlns:xacro="http://ros.org/wiki/xacro">
-  <xacro:include filename="$(find mir_description)/urdf/include/common_properties.urdf.xacro" />
-  <xacro:include filename="$(find mir_description)/urdf/include/imu.gazebo.urdf.xacro" />
-  <xacro:include filename="$(find mir_description)/urdf/include/mir_100.gazebo.xacro" />
-  <xacro:include filename="$(find mir_description)/urdf/include/mir_100.transmission.xacro" />
-  <xacro:include filename="$(find mir_description)/urdf/include/sick_s300.urdf.xacro" />
+  <xacro:include filename="$(find senai_models)/models/${model_class}/${model}/urdf/include/common_properties.urdf.xacro" />
+  <xacro:include filename="$(find senai_models)/models/${model_class}/${model}/urdf/include/imu.gazebo.urdf.xacro" />
+  <xacro:include filename="$(find senai_models)/models/${model_class}/${model}/urdf/include/mir_100.gazebo.xacro" />
+  <xacro:include filename="$(find senai_models)/models/${model_class}/${model}/urdf/include/mir_100.transmission.xacro" />
+  <xacro:include filename="$(find senai_models)/models/${model_class}/${model}/urdf/include/sick_s300.urdf.xacro" />
   <xacro:property name="deg_to_rad" value="0.017453293" />
   <xacro:property name="mir_100_base_mass" value="58.0" />
@@ -39,5 +39,5 @@
         <origin xyz="0 0 0" rpy="0 0 0" />
         <geometry>
-          <mesh filename="package://mir_description/meshes/visual/wheel.stl" />
+          <mesh filename="package://senai_models/models/${model_class}/${model}/meshes/visual/wheel.stl" />
         </geometry>
         <xacro:insert_block name="material_dark_grey" />
@@ -46,5 +46,5 @@
         <origin xyz="0 0 0" rpy="0 0 0" />
         <geometry>
-          <mesh filename="package://mir_description/meshes/visual/wheel.stl" />
+          <mesh filename="package://senai_models/models/${model_class}/${model}/meshes/visual/wheel.stl" />
         </geometry>
       </collision>
@@ -79,5 +79,5 @@
         <origin xyz="0 0 0" rpy="0 0 0" />
         <geometry>
-          <mesh filename="package://mir_description/meshes/visual/caster_wheel_base.stl" />
+          <mesh filename="package://senai_models/models/${model_class}/${model}/meshes/visual/caster_wheel_base.stl" />
         </geometry>
         <xacro:insert_block name="material_silver" />
@@ -86,5 +86,5 @@
         <origin xyz="0 0 0" rpy="0 0 0" />
         <geometry>
-          <mesh filename="package://mir_description/meshes/collision/caster_wheel_base.stl" />
+          <mesh filename="package://senai_models/models/${model_class}/${model}/meshes/collision/caster_wheel_base.stl" />
         </geometry>
       </collision>
@@ -107,5 +107,5 @@
         <origin xyz="0 0 0" rpy="0 0 0" />
         <geometry>
-          <mesh filename="package://mir_description/meshes/visual/wheel.stl" />
+          <mesh filename="package://senai_models/models/${model_class}/${model}/meshes/visual/wheel.stl" />
         </geometry>
         <xacro:insert_block name="material_dark_grey" />
@@ -114,5 +114,5 @@
         <origin xyz="0 0 0" rpy="0 0 0" />
         <geometry>
-          <mesh filename="package://mir_description/meshes/visual/wheel.stl" />
+          <mesh filename="package://senai_models/models/${model_class}/${model}/meshes/visual/wheel.stl" />
         </geometry>
       </collision>
@@ -136,5 +136,5 @@
         <origin xyz="${mir_100_act_wheel_dx} 0 0" rpy="0 0 0" />
         <geometry>
-          <mesh filename="package://mir_description/meshes/visual/mir_100_base.stl" />
+          <mesh filename="package://senai_models/models/${model_class}/${model}/meshes/visual/mir_100_base.stl" />
         </geometry>
         <xacro:insert_block name="material_white" />
@@ -143,5 +143,5 @@
         <origin xyz="${mir_100_act_wheel_dx} 0 0" rpy="0 0 0" />
         <geometry>
-          <mesh filename="package://mir_description/meshes/collision/mir_100_base.stl" />
+          <mesh filename="package://senai_models/models/${model_class}/${model}/meshes/collision/mir_100_base.stl" />
         </geometry>
       </collision>

File: models/robots/mir100/urdf/include/sick_s300.urdf.xacro (robot description, xacro)
@@ -1,5 +1,5 @@
 <?xml version="1.0"?>
 <robot xmlns:xacro="http://ros.org/wiki/xacro">
-  <xacro:include filename="$(find mir_description)/urdf/include/common_properties.urdf.xacro" />
+  <xacro:include filename="$(find senai_models)/models/${model_class}/${model}/urdf/include/common_properties.urdf.xacro" />
   <xacro:property name="laser_x" value="0.156" />
   <xacro:property name="laser_y" value="0.155" />
@@ -11,5 +11,5 @@
         <origin xyz="0.0 0.0 0.0" rpy="${pi} 0 0" />
         <geometry>
-          <mesh filename="package://mir_description/meshes/visual/sick_lms-100.stl" />
+          <mesh filename="package://senai_models/models/${model_class}/${model}/meshes/visual/sick_lms-100.stl" />
         </geometry>
         <!-- <xacro:insert_block name="material_yellow" /> -->
@@ -19,5 +19,5 @@
         <origin xyz="0.0 0.0 0.0" rpy="${pi} 0 0" />
         <geometry>
-          <mesh filename="package://mir_description/meshes/visual/sick_lms-100.stl" />
+          <mesh filename="package://senai_models/models/${model_class}/${model}/meshes/visual/sick_lms-100.stl" />
         </geometry>
       </collision>

File: models/robots/mir100/urdf/mir100.urdf.xacro (robot description, xacro)
@@ -1,8 +1,10 @@
 <?xml version="1.0"?>
-<robot xmlns:xacro="http://ros.org/wiki/xacro"
-       name="mir_100" >
+<robot xmlns:xacro="http://ros.org/wiki/xacro" name="$(arg model_name)" >
+  <xacro:arg name="model_name" default="bot" />
+  <xacro:property name="model_class" value="robots" />
+  <xacro:property name="model" value="mir100" />
   <!-- MiR100 base -->
-  <xacro:include filename="$(find mir_description)/urdf/include/mir_100_v1.urdf.xacro" />
-  <xacro:include filename="$(find mir_description)/urdf/include/common.gazebo.xacro" />
+  <xacro:include filename="$(find senai_models)/models/${model_class}/${model}/urdf/include/mir_100_v1.urdf.xacro" />
+  <xacro:include filename="$(find senai_models)/models/${model_class}/${model}/urdf/include/common.gazebo.xacro" />
   <xacro:arg name="tf_prefix" default="" />
   <xacro:property name="tf_prefix_" value="$(arg tf_prefix)" />

Commit message: adding lidar topics

File: models/robots/mir100/urdf/include/mir_100_v1.urdf.xacro (robot description, xacro)
@@ -3,5 +3,5 @@
   <xacro:include filename="$(find senai_models)/models/${model_class}/${model}/urdf/include/common_properties.urdf.xacro" />
   <xacro:include filename="$(find senai_models)/models/${model_class}/${model}/urdf/include/imu.gazebo.urdf.xacro" />
-  <!-- <xacro:include filename="$(find senai_models)/models/${model_class}/${model}/urdf/include/mir_100.gazebo.xacro" /> -->
+  <xacro:include filename="$(find senai_models)/models/${model_class}/${model}/urdf/include/mir_100.gazebo.xacro" />
   <xacro:include filename="$(find senai_models)/models/${model_class}/${model}/urdf/include/mir_100.transmission.xacro" />
   <xacro:include filename="$(find senai_models)/models/${model_class}/${model}/urdf/include/sick_s300.urdf.xacro" />
@@ -210,5 +210,5 @@
     <!-- set the gazebo friction parameters for the wheels -->
     <xacro:set_all_wheel_frictions prefix="${prefix}"/>
-    <xacro:p3d_base_controller prefix="${prefix}" />
+    <!-- <xacro:p3d_base_controller prefix="${prefix}" /> -->
   </xacro:macro>
 </robot>

File: models/robots/mir100/urdf/include/sick_s300.urdf.xacro (robot description, xacro)
@@ -29,46 +29,7 @@
       <!-- <material value="Gazebo/Yellow" /> -->
       <material value="Gazebo/FlatBlack" />
-      <sensor name="${prefix}${link}" type='lidar'>
+      <sensor type="ray" name="${prefix}${link}">
         <pose>0 0 0 0 0 0</pose>
-        <visualize>true</visualize>
-        <update_rate>12.5</update_rate>
-        <lidar>
-            <scan>
-                <horizontal>
-                    <samples>541</samples>
-                    <resolution>1</resolution>
-                    <min_angle>-2.35619449615</min_angle>
-                    <max_angle>2.35619449615</max_angle>
-                </horizontal>
-            </scan>
-            <range>
-                <min>0.05</min>
-                <max>29.0</max>
-                <resolution>0.01</resolution>
-            </range>
-            <noise>
-              <type>gaussian</type>
-              <!-- Noise parameters based on published spec for S300 achieving
-                  "+-29mm" accuracy at range < 3m (~0.01 of the range) at
-                  1 sigma. -->
-              <mean>0.0</mean>
-              <stddev>0.01</stddev>
-            </noise>
-        </lidar>
-        <xacro:if value="${gazebo_version == 'classic'}">
-          <plugin name="gazebo_ros_${link}_controller" filename="libgazebo_ros_laser.so">
-            <frameName>${prefix}${link}</frameName>
-            <topicName>${topic}</topicName>
-          </plugin>
-        </xacro:if>
-        <xacro:if value="${gazebo_version == 'ignition'}">
-          <plugin filename="libignition-gazebo-sensors-system.so" name="ignition::gazebo::systems::Sensors">
-            <render_engine>ogre2</render_engine>
-          </plugin>
-        </xacro:if>
-      </sensor>
-      <!-- <sensor type="ray" name="${prefix}${link}">
-        <pose>0 0 0 0 0 0</pose>
-        <visualize>true</visualize>
+        <visualize>false</visualize>
         <update_rate>12.5</update_rate>
         <ray>
@@ -76,5 +37,5 @@
             <horizontal>
               <samples>541</samples>
-              <resolution>1</resolution>  <!- has to be 1; actual resolution will be computed from number of samples + min_angle/max_angle ->
+              <resolution>1</resolution>  <!-- has to be 1; actual resolution will be computed from number of samples + min_angle/max_angle -->
               <min_angle>-2.35619449615</min_angle>
               <max_angle>2.35619449615</max_angle>
@@ -88,7 +49,7 @@
           <noise>
             <type>gaussian</type>
-            <!- Noise parameters based on published spec for S300 achieving
+            <!-- Noise parameters based on published spec for S300 achieving
                  "+-29mm" accuracy at range < 3m (~0.01 of the range) at
-                 1 sigma. ->
+                 1 sigma. -->
             <mean>0.0</mean>
             <stddev>0.01</stddev>
@@ -96,10 +57,20 @@
         </ray>
         <xacro:if value="${gazebo_version == 'classic'}">
-          <plugin name="gazebo_ros_${link}_controller" filename="libgazebo_ros_laser.so">
-            <frameName>${prefix}${link}</frameName>
-            <topicName>${topic}</topicName>
+          <xacro:property name="sensor_name" value="${link.replace('_link','')}"/>
+          <plugin name="lidar_sensor_broadcaster_${sensor_name}" filename="libgazebo_ros_ray_sensor.so">
+            <ros>
+              <namespace>/$(arg model_name)/lidar_sensor_broadcaster</namespace>
+              <remapping>lidar_sensor_broadcaster_${sensor_name}/out:=${sensor_name}/scan</remapping>
+            </ros>
+            <output_type>sensor_msgs/LaserScan</output_type>
+            <frame_name>${prefix}${link}</frame_name>
           </plugin>
         </xacro:if>
-      </sensor> -->
+        <xacro:if value="${gazebo_version == 'ignition'}">
+          <plugin filename="libignition-gazebo-sensors-system.so" name="ignition::gazebo::systems::Sensors">
+            <render_engine>ogre2</render_engine>
+          </plugin>
+        </xacro:if>
+      </sensor>
     </gazebo>
   </xacro:macro>
