Commit message: fixing frames and adding ultrasound sensor

File: models/robots/mir100/urdf/include/mir_100.gazebo.xacro (robot description, xacro)
@@ -4,23 +4,21 @@
     <gazebo>
       <xacro:if value="${gazebo_version == 'classic'}">
-        <plugin name="diff_drive_controller" filename="libgazebo_ros_diff_drive.so">
-          <legacyMode>false</legacyMode>
-          <alwaysOn>true</alwaysOn>
-          <updateRate>1000.0</updateRate>
-          <leftJoint>${left_wheel_joint}</leftJoint>
-          <rightJoint>${right_wheel_joint}</rightJoint>
-          <wheelSeparation>${wheel_separation}</wheelSeparation>
-          <wheelDiameter>${2*wheel_radius}</wheelDiameter>
-          <wheelTorque>10</wheelTorque>
-          <publishTf>1</publishTf>
-          <odometryFrame>map</odometryFrame>
-          <commandTopic>/model/$(arg model_name)/cmd_vel</commandTopic>
-          <odometryTopic>/model/$(arg model_name)/odom</odometryTopic>
-          <robotBaseFrame>base_footprint</robotBaseFrame>
-          <wheelAcceleration>2.8</wheelAcceleration>
-          <publishWheelJointState>true</publishWheelJointState>
-          <publishWheelTF>false</publishWheelTF>
-          <odometrySource>world</odometrySource>
-          <rosDebugLevel>Debug</rosDebugLevel>
+        <plugin name="diff_drive" filename="libgazebo_ros_diff_drive.so">
+          <!-- <legacyMode>false</legacyMode>
+          <alwaysOn>true</alwaysOn> -->
+          <!-- <update_rate>60.0</update_rate> -->
+          <left_joint>${left_wheel_joint}</left_joint>
+          <right_joint>${right_wheel_joint}</right_joint>
+          <wheel_separation>${wheel_separation}</wheel_separation>
+          <wheel_diameter>${2*wheel_radius}</wheel_diameter>
+          <max_wheel_torque>10</max_wheel_torque>
+          <max_wheel_acceleration>2.8</max_wheel_acceleration>
+          <odometry_frame>odom</odometry_frame>
+          <robot_base_frame>base_footprint</robot_base_frame>
+          <publish_odom>true</publish_odom>
+          <publish_odom_tf>true</publish_odom_tf>
+          <publish_wheel_tf>true</publish_wheel_tf>
+          <!-- <topic>/model/$(arg model_name)/cmd_vel</topic>
+          <odom_topic>/model/$(arg model_name)/odom</odom_topic> -->
         </plugin>
       </xacro:if>

File: models/robots/mir100/urdf/include/mir_100_v1.urdf.xacro (robot description, xacro)
@@ -6,4 +6,5 @@
   <xacro:include filename="$(find senai_models)/models/${model_class}/${model}/urdf/include/mir_100.transmission.xacro" />
   <xacro:include filename="$(find senai_models)/models/${model_class}/${model}/urdf/include/sick_s300.urdf.xacro" />
+  <xacro:include filename="$(find senai_models)/models/${model_class}/${model}/urdf/include/ultrasound.urdf.xacro" />
   <xacro:property name="deg_to_rad" value="0.017453293" />
   <xacro:property name="mir_100_base_mass" value="58.0" />
@@ -181,16 +182,6 @@
     <xacro:sick_s300 prefix="${prefix}" link="back_laser_link" topic="b_scan" />
     <!-- Ultrasound sensors -->
-    <joint name="${prefix}us_1_joint" type="fixed">   <!-- right ultrasound -->
-      <parent link="${prefix}base_link" />
-      <child link="${prefix}us_1_frame" />
-      <origin xyz="0.45 -0.12 0.16 " rpy="0 0 0" />  <!-- from visually matching to the mesh of the MiR -->
-    </joint>
-    <link name="${prefix}us_1_frame" />
-    <joint name="${prefix}us_2_joint" type="fixed">   <!-- left ultrasound -->
-      <parent link="${prefix}base_link" />
-      <child link="${prefix}us_2_frame" />
-      <origin xyz="0.45 0.12 0.16 " rpy="0 0 0" />  <!-- from visually matching to the mesh of the MiR -->
-    </joint>
-    <link name="${prefix}us_2_frame" />
+    <xacro:ultrasound_hcsr04 side="right" orientation="-1" prefix="${prefix}"/>
+    <xacro:ultrasound_hcsr04 side="left" orientation="1" prefix="${prefix}"/>
     <!-- wheels -->
     <xacro:actuated_wheel prefix="${prefix}" locationprefix="left" locationright="-1"/>

File: models/robots/mir100/urdf/include/sick_s300.urdf.xacro (robot description, xacro)
@@ -58,8 +58,8 @@
         <xacro:if value="${gazebo_version == 'classic'}">
           <xacro:property name="sensor_name" value="${link.replace('_link','')}"/>
-          <plugin name="lidar_sensor_broadcaster_${sensor_name}" filename="libgazebo_ros_ray_sensor.so">
+          <plugin name="${sensor_name}" filename="libgazebo_ros_ray_sensor.so">
             <ros>
               <namespace>/$(arg model_name)/lidar_sensor_broadcaster</namespace>
-              <remapping>lidar_sensor_broadcaster_${sensor_name}/out:=${sensor_name}/scan</remapping>
+              <remapping>${sensor_name}/out:=${sensor_name}/scan</remapping>
             </ros>
             <output_type>sensor_msgs/LaserScan</output_type>

File: models/robots/mir100/urdf/mir100.urdf.xacro (robot description, xacro)
@@ -32,5 +32,5 @@
         <plugin>gazebo_ros2_control/GazeboSystem</plugin>
       </hardware>
-      <joint name="left_wheel_joint">
+      <joint name="${prefix}left_wheel_joint">
         <command_interface name="velocity">
             <param name="min">-10</param>
@@ -40,5 +40,5 @@
         <state_interface name="velocity" />
       </joint>
-      <joint name="right_wheel_joint">
+      <joint name="${prefix}right_wheel_joint">
           <command_interface name="velocity">
               <param name="min">-10</param>
@@ -75,5 +75,5 @@
         <plugin>ign_ros2_control/IgnitionSystem</plugin>
       </hardware>
-      <joint name="left_wheel_joint">
+      <joint name="${prefix}left_wheel_joint">
         <command_interface name="velocity">
             <param name="min">-10</param>
@@ -83,5 +83,5 @@
         <state_interface name="velocity" />
       </joint>
-      <joint name="right_wheel_joint">
+      <joint name="${prefix}right_wheel_joint">
           <command_interface name="velocity">
               <param name="min">-10</param>
