Commit message: fixing joints

File: models/robots/mir100/urdf/include/mir_100.transmission.xacro (robot description, xacro)
@@ -4,5 +4,6 @@
     <transmission name="${prefix}${locationprefix}_wheel_trans">
       <type>transmission_interface/SimpleTransmission</type>
-      <joint name="${prefix}${locationprefix}_wheel_joint">
+      <!-- <joint name="${prefix}${locationprefix}_wheel_joint"> -->
+      <joint name="${locationprefix}_wheel_joint">
         <hardwareInterface>hardware_interface/VelocityJointInterface</hardwareInterface>
       </joint>

File: models/robots/mir100/urdf/include/mir_100_v1.urdf.xacro (robot description, xacro)
@@ -26,11 +26,4 @@
   <xacro:property name="imu_stdev" value="0.00017" />
   <xacro:macro name="actuated_wheel" params="prefix locationprefix locationright">
-    <joint name="${prefix}${locationprefix}_wheel_joint" type="continuous">
-      <origin xyz="0.0 ${-mir_100_act_wheel_dy * locationright} ${mir_100_act_wheel_radius}" rpy="0 0 0" />
-      <parent link="${prefix}base_link" />
-      <child link="${prefix}${locationprefix}_wheel_link" />
-      <axis xyz="0 1 0" />
-      <limit effort="100" velocity="20.0" />
-    </joint>
     <link name="${prefix}${locationprefix}_wheel_link">
       <xacro:cylinder_inertial mass="${mir_100_act_wheel_mass}" radius="${mir_100_act_wheel_radius}" length="${mir_100_act_wheel_width}">
@@ -51,4 +44,12 @@
       </collision>
     </link>
+    <!-- <joint name="${prefix}${locationprefix}_wheel_joint" type="continuous"> -->
+    <joint name="${locationprefix}_wheel_joint" type="continuous">
+      <origin xyz="0.0 ${-mir_100_act_wheel_dy * locationright} ${mir_100_act_wheel_radius}" rpy="0 0 0" />
+      <parent link="${prefix}base_link" />
+      <child link="${prefix}${locationprefix}_wheel_link" />
+      <axis xyz="0 1 0" />
+      <limit effort="100" velocity="20.0" />
+    </joint>
     <gazebo reference="${prefix}${locationprefix}_wheel_link">
       <material>Gazebo/DarkGrey</material>
@@ -56,12 +57,4 @@
   </xacro:macro>
   <xacro:macro name="caster_wheel" params="prefix locationprefix locationright wheel_base_dx">
-    <!-- caster hub -->
-    <joint name="${prefix}${locationprefix}_caster_rotation_joint" type="continuous">
-      <origin xyz="${wheel_base_dx} ${-mir_100_caster_wheel_base_dy * locationright} ${mir_100_caster_wheel_base_dz}" rpy="0 0 0" />
-      <parent link="${prefix}base_link" />
-      <child link="${prefix}${locationprefix}_caster_rotation_link" />
-      <axis xyz="0 0 1" />
-      <dynamics damping="0.01" friction="0.0"/>
-    </joint>
     <link name="${prefix}${locationprefix}_caster_rotation_link">
       <inertial>
@@ -91,8 +84,34 @@
       </collision>
     </link>
+    <!-- caster hub -->
+    <joint name="${prefix}${locationprefix}_caster_rotation_joint" type="continuous">
+      <origin xyz="${wheel_base_dx} ${-mir_100_caster_wheel_base_dy * locationright} ${mir_100_caster_wheel_base_dz}" rpy="0 0 0" />
+      <parent link="${prefix}base_link" />
+      <child link="${prefix}${locationprefix}_caster_rotation_link" />
+      <axis xyz="0 0 1" />
+      <dynamics damping="0.01" friction="0.0"/>
+    </joint>
     <gazebo reference="${prefix}${locationprefix}_caster_rotation_link">
       <material>Gazebo/Grey</material>
     </gazebo>
     <!-- caster wheel -->
+    <link name="${prefix}${locationprefix}_caster_wheel_link">
+      <xacro:cylinder_inertial mass="${mir_100_caster_wheel_mass}" radius="${mir_100_caster_wheel_radius}" length="${mir_100_caster_wheel_width}">
+        <origin xyz="0 0 0" rpy="${0.5 * pi} 0 0" />
+      </xacro:cylinder_inertial>
+      <visual>
+        <origin xyz="0 0 0" rpy="0 0 0" />
+        <geometry>
+          <mesh filename="package://senai_models/models/${model_class}/${model}/meshes/visual/wheel.stl" />
+        </geometry>
+        <xacro:insert_block name="material_dark_grey" />
+      </visual>
+      <collision>
+        <origin xyz="0 0 0" rpy="0 0 0" />
+        <geometry>
+          <mesh filename="package://senai_models/models/${model_class}/${model}/meshes/visual/wheel.stl" />
+        </geometry>
+      </collision>
+    </link>
     <joint name="${prefix}${locationprefix}_caster_wheel_joint" type="continuous">
       <origin xyz="${mir_100_caster_wheel_dx} ${-mir_100_caster_wheel_dy * locationright} ${mir_100_caster_wheel_dz}" rpy="0 0 0" />
@@ -101,22 +120,4 @@
       <axis xyz="0 1 0" />
     </joint>
-    <link name="${prefix}${locationprefix}_caster_wheel_link">
-      <xacro:cylinder_inertial mass="${mir_100_caster_wheel_mass}" radius="${mir_100_caster_wheel_radius}" length="${mir_100_caster_wheel_width}">
-        <origin xyz="0 0 0" rpy="${0.5 * pi} 0 0" />
-      </xacro:cylinder_inertial>
-      <visual>
-        <origin xyz="0 0 0" rpy="0 0 0" />
-        <geometry>
-          <mesh filename="package://senai_models/models/${model_class}/${model}/meshes/visual/wheel.stl" />
-        </geometry>
-        <xacro:insert_block name="material_dark_grey" />
-      </visual>
-      <collision>
-        <origin xyz="0 0 0" rpy="0 0 0" />
-        <geometry>
-          <mesh filename="package://senai_models/models/${model_class}/${model}/meshes/visual/wheel.stl" />
-        </geometry>
-      </collision>
-    </link>
     <gazebo reference="${prefix}${locationprefix}_caster_wheel_link">
       <material>Gazebo/DarkGrey</material>

File: models/robots/mir100/urdf/mir100.urdf.xacro (robot description, xacro)
@@ -32,5 +32,6 @@
         <plugin>gazebo_ros2_control/GazeboSystem</plugin>
       </hardware>
-      <joint name="${prefix}left_wheel_joint">
+      <!-- <joint name="${prefix}left_wheel_joint"> -->
+      <joint name="left_wheel_joint">
         <command_interface name="velocity">
             <param name="min">-10</param>
@@ -40,5 +41,6 @@
         <state_interface name="velocity" />
       </joint>
-      <joint name="${prefix}right_wheel_joint">
+      <!-- <joint name="${prefix}right_wheel_joint"> -->
+      <joint name="right_wheel_joint">
           <command_interface name="velocity">
               <param name="min">-10</param>
@@ -75,5 +77,6 @@
         <plugin>ign_ros2_control/IgnitionSystem</plugin>
       </hardware>
-      <joint name="${prefix}left_wheel_joint">
+      <!-- <joint name="${prefix}left_wheel_joint"> -->
+      <joint name="left_wheel_joint">
         <command_interface name="velocity">
             <param name="min">-10</param>
@@ -83,5 +86,6 @@
         <state_interface name="velocity" />
       </joint>
-      <joint name="${prefix}right_wheel_joint">
+      <!-- <joint name="${prefix}right_wheel_joint"> -->
+      <joint name="right_wheel_joint">
           <command_interface name="velocity">
               <param name="min">-10</param>
@@ -108,4 +112,5 @@
         <ros>
           <namespace>/$(arg model_name)</namespace>
+          <remapping>/$(arg model_name)/joint_states:=/joint_state_broadcaster/joint_states</remapping>
         </ros>
         <parameters>$(find senai_models)/models/${model_class}/${model}/config/$(arg gazebo_version)/${model}_controllers.yaml</parameters>
