Commit message: adding lidar sensor broadcaster and tf topics

File: models/robots/mir100/files/MiR100.urdf (robot description, URDF)
Before this commit: robot mir100, 19 links, 18 joints
Links:
- removed link us_1_frame
- removed link us_2_frame
- added link camera_link; visual box size=0.010 0.03 0.03
- added link camera_link_optical
- added link us_left_frame
- added link us_right_frame
Joints:
- removed joint us_1_joint
- removed joint us_2_joint
- added joint camera_joint: type fixed, parent base_link, child camera_link, origin xyz=0.45 0.039 0.279 rpy=0 0 0
- added joint camera_optical_joint: type fixed, parent camera_link, child camera_link_optical, origin xyz=0 0 0 rpy=-1.5707963267948966 0 -1.5707963267948966
- added joint us_left_joint: type fixed, parent base_link, child us_left_frame, origin xyz=0.45 0.12 0.16  rpy=0 0 0
- added joint us_right_joint: type fixed, parent base_link, child us_right_frame, origin xyz=0.45 -0.12 0.16  rpy=0 0 0

File: models/robots/mir100/urdf/include/imu.gazebo.urdf.xacro (robot description, xacro)
@@ -18,13 +18,13 @@
         <visualize>true</visualize>
         <topic>/model/$(arg model_name)/imu_data</topic>
-        <plugin filename="ignition-gazebo-imu-system" name="gz::sim::systems::Imu">
+        <!-- <plugin filename="ignition-gazebo-imu-system" name="gz::sim::systems::Imu">
           <topicName>${imu_topic}</topicName>
           <bodyName>${link}</bodyName>
-          <updateRateHZ>${update_rate}</updateRateHZ>  <!-- this is the publish rate -->
+          <updateRateHZ>${update_rate}</updateRateHZ>  <!- this is the publish rate ->
           <gaussianNoise>${stdev * stdev}</gaussianNoise>
           <xyzOffset>0 0 0</xyzOffset>
           <rpyOffset>0 0 0</rpyOffset>
-          <frameName>${imu_frame}</frameName>  <!-- from real MiR -->
-        </plugin>
+          <frameName>${imu_frame}</frameName>  <!- from real MiR ->
+        </plugin> -->
         <pose>0 0 0 0 0 0</pose>
       </sensor>

File: models/robots/mir100/urdf/include/sick_s300.urdf.xacro (robot description, xacro)
@@ -36,5 +36,5 @@
           <scan>
             <horizontal>
-              <samples>541</samples>
+              <samples>684</samples>
               <resolution>1</resolution>  <!-- has to be 1; actual resolution will be computed from number of samples + min_angle/max_angle -->
               <min_angle>-2.35619449615</min_angle>

Commit message: Adding range_sensor and image_raw topics

File: models/robots/mir100/files/MiR100.urdf (robot description, URDF)
Before this commit: robot MiR100, 21 links, 20 joints
Links:
- removed link back_laser_link
- removed link base_footprint
- removed link base_link
- removed link bl_caster_rotation_link
- removed link bl_caster_wheel_link
- removed link br_caster_rotation_link
- removed link br_caster_wheel_link
- removed link camera_link
- removed link camera_link_optical
- removed link fl_caster_rotation_link
- removed link fl_caster_wheel_link
- removed link fr_caster_rotation_link
- removed link fr_caster_wheel_link
- removed link front_laser_link
- removed link imu_frame
- removed link imu_link
- removed link left_wheel_link
- removed link right_wheel_link
- removed link surface
- removed link us_left_frame
- removed link us_right_frame
- added link MiR100/back_laser_link, mass 2.0; collision mesh filename=package://senai_models/models/robots/mir100/meshes/visual/s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; visual mesh filename=package://senai_models/models/robots/mir100/meshes/visual/s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
- added link MiR100/base_footprint
- added link MiR100/base_link, mass 58.0; collision mesh filename=package://senai_models/models/robots/mir100/meshes/collisio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; visual mesh filename=package://senai_models/models/robots/mir100/meshes/visual/m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
- added link MiR100/bl_caster_rotation_link, mass 0.3097539019; collision mesh filename=package://senai_models/models/robots/mir100/meshes/collisio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; visual mesh filename=package://senai_models/models/robots/mir100/meshes/visual/c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
- added link MiR100/bl_caster_wheel_link, mass 1.0; collision mesh filename=package://senai_models/models/robots/mir100/meshes/visual/w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; visual mesh filename=package://senai_models/models/robots/mir100/meshes/visual/w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
- added link MiR100/br_caster_rotation_link, mass 0.3097539019; collision mesh filename=package://senai_models/models/robots/mir100/meshes/collisio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; visual mesh filename=package://senai_models/models/robots/mir100/meshes/visual/c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
- added link MiR100/br_caster_wheel_link, mass 1.0; collision mesh filename=package://senai_models/models/robots/mir100/meshes/visual/w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; visual mesh filename=package://senai_models/models/robots/mir100/meshes/visual/w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
- added link MiR100/camera_link; visual box size=0.010 0.03 0.03
- added link MiR100/camera_link_optical
- added link MiR100/fl_caster_rotation_link, mass 0.3097539019; collision mesh filename=package://senai_models/models/robots/mir100/meshes/collisio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; visual mesh filename=package://senai_models/models/robots/mir100/meshes/visual/c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
- added link MiR100/fl_caster_wheel_link, mass 1.0; collision mesh filename=package://senai_models/models/robots/mir100/meshes/visual/w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; visual mesh filename=package://senai_models/models/robots/mir100/meshes/visual/w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
- added link MiR100/fr_caster_rotation_link, mass 0.3097539019; collision mesh filename=package://senai_models/models/robots/mir100/meshes/collisio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; visual mesh filename=package://senai_models/models/robots/mir100/meshes/visual/c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
- added link MiR100/fr_caster_wheel_link, mass 1.0; collision mesh filename=package://senai_models/models/robots/mir100/meshes/visual/w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; visual mesh filename=package://senai_models/models/robots/mir100/meshes/visual/w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
- added link MiR100/front_laser_link, mass 2.0; collision mesh filename=package://senai_models/models/robots/mir100/meshes/visual/s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; visual mesh filename=package://senai_models/models/robots/mir100/meshes/visual/s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
- added link MiR100/imu_frame
- added link MiR100/imu_link
- added link MiR100/left_wheel_link, mass 1.0; collision mesh filename=package://senai_models/models/robots/mir100/meshes/visual/w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; visual mesh filename=package://senai_models/models/robots/mir100/meshes/visual/w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
- added link MiR100/right_wheel_link, mass 1.0; collision mesh filename=package://senai_models/models/robots/mir100/meshes/visual/w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; visual mesh filename=package://senai_models/models/robots/mir100/meshes/visual/w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
- added link MiR100/surface
- added link MiR100/us_left_frame
- added link MiR100/us_right_frame
Joints:
- removed joint base_joint
- removed joint base_link_surface_joint
- removed joint base_link_to_back_laser_joint
- removed joint base_link_to_front_laser_joint
- removed joint base_link_to_imu_joint
- removed joint bl_caster_rotation_joint
- removed joint bl_caster_wheel_joint
- removed joint br_caster_rotation_joint
- removed joint br_caster_wheel_joint
- removed joint camera_joint
- removed joint camera_optical_joint
- removed joint fl_caster_rotation_joint
- removed joint fl_caster_wheel_joint
- removed joint fr_caster_rotation_joint
- removed joint fr_caster_wheel_joint
- removed joint imu_link_to_imu_frame_joint
- removed joint us_left_joint
- removed joint us_right_joint
- added joint MiR100/base_joint: type fixed, parent MiR100/base_footprint, child MiR100/base_link, origin xyz=0 0 0 rpy=0 0 0
- added joint MiR100/base_link_surface_joint: type fixed, parent MiR100/base_link, child MiR100/surface, origin xyz=0.037646 0 0.352 rpy=0 0 0, axis 0 0 1
- added joint MiR100/base_link_to_back_laser_joint: type fixed, parent MiR100/base_link, child MiR100/back_laser_link, origin xyz=-0.3548 -0.2352 0.1914 rpy=0.0 0.0 -2.356194490192345
- added joint MiR100/base_link_to_front_laser_joint: type fixed, parent MiR100/base_link, child MiR100/front_laser_link, origin xyz=0.4288 0.2358 0.1914 rpy=0.0 0.0 0.7853981633974483
- added joint MiR100/base_link_to_imu_joint: type fixed, parent MiR100/base_link, child MiR100/imu_link, origin xyz=0.0 0.0 0.25 rpy=0 0 0
- added joint MiR100/bl_caster_rotation_joint: type continuous, parent MiR100/base_link, child MiR100/bl_caster_rotation_link, origin xyz=-0.270154 0.203 0.1565 rpy=0 0 0, axis 0 0 1
- added joint MiR100/bl_caster_wheel_joint: type continuous, parent MiR100/bl_caster_rotation_link, child MiR100/bl_caster_wheel_link, origin xyz=-0.0382 0 -0.094 rpy=0 0 0, axis 0 1 0
- added joint MiR100/br_caster_rotation_joint: type continuous, parent MiR100/base_link, child MiR100/br_caster_rotation_link, origin xyz=-0.270154 -0.203 0.1565 rpy=0 0 0, axis 0 0 1
- added joint MiR100/br_caster_wheel_joint: type continuous, parent MiR100/br_caster_rotation_link, child MiR100/br_caster_wheel_link, origin xyz=-0.0382 0 -0.094 rpy=0 0 0, axis 0 1 0
- added joint MiR100/camera_joint: type fixed, parent MiR100/base_link, child MiR100/camera_link, origin xyz=0.45 0.039 0.279 rpy=0 0 0
- added joint MiR100/camera_optical_joint: type fixed, parent MiR100/camera_link, child MiR100/camera_link_optical, origin xyz=0 0 0 rpy=-1.5707963267948966 0 -1.5707963267948966
- added joint MiR100/fl_caster_rotation_joint: type continuous, parent MiR100/base_link, child MiR100/fl_caster_rotation_link, origin xyz=0.341346 0.203 0.1565 rpy=0 0 0, axis 0 0 1
- added joint MiR100/fl_caster_wheel_joint: type continuous, parent MiR100/fl_caster_rotation_link, child MiR100/fl_caster_wheel_link, origin xyz=-0.0382 0 -0.094 rpy=0 0 0, axis 0 1 0
- added joint MiR100/fr_caster_rotation_joint: type continuous, parent MiR100/base_link, child MiR100/fr_caster_rotation_link, origin xyz=0.341346 -0.203 0.1565 rpy=0 0 0, axis 0 0 1
- added joint MiR100/fr_caster_wheel_joint: type continuous, parent MiR100/fr_caster_rotation_link, child MiR100/fr_caster_wheel_link, origin xyz=-0.0382 0 -0.094 rpy=0 0 0, axis 0 1 0
- added joint MiR100/imu_link_to_imu_frame_joint: type fixed, parent MiR100/imu_link, child MiR100/imu_frame, origin xyz=0 0 0 rpy=0 0 0
- added joint MiR100/us_left_joint: type fixed, parent MiR100/base_link, child MiR100/us_left_frame, origin xyz=0.45 0.12 0.16  rpy=0 0 0
- added joint MiR100/us_right_joint: type fixed, parent MiR100/base_link, child MiR100/us_right_frame, origin xyz=0.45 -0.12 0.16  rpy=0 0 0
- joint left_wheel_joint: child left_wheel_link -> MiR100/left_wheel_link; parent base_link -> MiR100/base_link
- joint right_wheel_joint: child right_wheel_link -> MiR100/right_wheel_link; parent base_link -> MiR100/base_link
